Commit message: repair urdf

File: foxy_moveit2/cr3a_description/urdf/cr3a.xacro (robot description, xacro)
@@ -69,5 +69,5 @@
     <child link="Link1" />
     <axis xyz="0 0 1" />
-    <limit lower="-3.14" upper="3.14" effort="300" velocity="100" />
+    <limit lower="-3.14" upper="3.14" effort="0" velocity="0" />
   </joint>
   <link name="Link1">
@@ -115,5 +115,5 @@
     <child link="Link2" />
     <axis xyz="0 0 1" />
-    <limit lower="-1.57" upper="1.57" effort="300" velocity="100" />
+    <limit lower="-1.57" upper="1.57" effort="0" velocity="0" />
   </joint>
   <link name="Link2">
@@ -161,5 +161,5 @@
     <child link="Link3" />
     <axis xyz="0 0 1" />
-    <limit lower="-2.55" upper="2.55" effort="300" velocity="100" />
+    <limit lower="-2.55" upper="2.55" effort="0" velocity="0" />
   </joint>
   <link name="Link3">
@@ -207,5 +207,5 @@
     <child link="Link4" />
     <axis xyz="0 0 1" />
-    <limit lower="-3.14" upper="3.14" effort="300" velocity="100" />
+    <limit lower="-3.14" upper="3.14" effort="0" velocity="0" />
   </joint>
   <link name="Link4">
@@ -253,5 +253,5 @@
     <child link="Link5" />
     <axis xyz="0 0 1" />
-    <limit lower="-3.14" upper="3.14" effort="300" velocity="100" />
+    <limit lower="-3.14" upper="3.14" effort="0" velocity="0" />
   </joint>
   <link name="Link5">
@@ -299,5 +299,5 @@
     <child link="Link6" />
     <axis xyz="0 0 1" />
-    <limit lower="-3.14" upper="3.14" effort="300" velocity="100" />
+    <limit lower="-3.14" upper="3.14" effort="0" velocity="0" />
   </joint>
   <link name="Link6">
