Commit message: manual diffbot sim hil good

File: wmx_ros2_control/urdf/diffbot.wmx.urdf.xacro (robot description, xacro)
@@ -6,10 +6,4 @@
   <xacro:include filename="$(find movensys_navigation_description)/urdf/diffbot/perception.xacro"/>
   <xacro:include filename="$(find wmx_ros2_control)/urdf/diffbot.wmx.ros2_control.xacro"/>
-  <link name="base_footprint"/>
-  <joint name="base_link_joint" type="fixed">
-    <origin xyz="0 0 0.095" rpy="0 0 0"/>
-    <parent link="base_footprint"/>
-    <child link="base_link"/>
-  </joint>
   <xacro:diffbot/>
   <xacro:diffbot_wmx_ros2_control wmx_param_file="$(arg wmx_param_file)"/>
