Commit message: enable cyclic-buffer position streaming on cr3a

File: wmx_r2_control/urdf/cr3a.wmx.ros2_control.xacro (robot description, xacro)
@@ -1,7 +1,28 @@
 <?xml version="1.0"?>
 <robot xmlns:xacro="http://www.ros.org/wiki/xacro">
+  <!--
+    ros2_control description for the Dobot CR3A arm on WMX3.
+    stream_position:
+      true  - each joint exports a 'position' command interface, which
+              WmxSystemHardware streams to the servos through the WMX3 cyclic
+              buffer. This is what lets a standard JointTrajectoryController (and
+              therefore MoveIt Servo) drive the arm.
+      false - joints are feedback-only, as before. Motion must then come from the
+              standalone wmx_r2_package/joint_trajectory_controller node. Use
+              this to fall back without editing any files:
+                  ros2 launch wmx_r2_control wmx_r2_control_cr3a_manipulator.launch.py \
+                       stream_position:=false
+    cyclic_max_acc is a *trip*, not a limiter: exceeding it quick-stops the axis
+    and clears the buffer. joint_limits.yaml allows 2.0 rad/s^2, so 5.0 leaves
+    headroom. Raise it first if you see MaxAccError during normal motion.
+  -->
   <xacro:macro name="movensys_manipulator_arm_wmx_r2_control"
                params="name:=WmxManipulatorArmSystem
-                       wmx_param_file">
+                       wmx_param_file
+                       stream_position:=true
+                       cyclic_max_acc:=5.0
+                       cyclic_target_periods:=2
+                       cyclic_push_period_ms:=10.0
+                       cyclic_buffer_horizon_s:=5.0">
     <ros2_control name="${name}" type="system">
       <hardware>
@@ -9,18 +30,28 @@
         <param name="device_name">wmx_cr3a_control</param>
         <param name="wmx_param_file">${wmx_param_file}</param>
+        <!-- Seed for the write() period. The hardware measures the real period
+             and converges on it, so this only has to be close; keep it equal to
+             1000 / controller_manager update_rate in cr3a_controllers.yaml. -->
+        <param name="cyclic_push_period_ms">${cyclic_push_period_ms}</param>
+        <param name="cyclic_target_periods">${cyclic_target_periods}</param>
+        <param name="cyclic_max_acc">${cyclic_max_acc}</param>
+        <param name="cyclic_buffer_horizon_s">${cyclic_buffer_horizon_s}</param>
       </hardware>
-      <xacro:macro name="arm_joint" params="joint axis">
+      <xacro:macro name="arm_joint" params="joint axis stream">
         <joint name="${joint}">
           <param name="axis">${axis}</param>
+          <xacro:if value="${stream}">
+            <command_interface name="position"/>
+          </xacro:if>
           <state_interface name="position"/>
           <state_interface name="velocity"/>
         </joint>
       </xacro:macro>
-      <xacro:arm_joint joint="joint1" axis="0"/>
-      <xacro:arm_joint joint="joint2" axis="1"/>
-      <xacro:arm_joint joint="joint3" axis="2"/>
-      <xacro:arm_joint joint="joint4" axis="3"/>
-      <xacro:arm_joint joint="joint5" axis="4"/>
-      <xacro:arm_joint joint="joint6" axis="5"/>
+      <xacro:arm_joint joint="joint1" axis="0" stream="${stream_position}"/>
+      <xacro:arm_joint joint="joint2" axis="1" stream="${stream_position}"/>
+      <xacro:arm_joint joint="joint3" axis="2" stream="${stream_position}"/>
+      <xacro:arm_joint joint="joint4" axis="3" stream="${stream_position}"/>
+      <xacro:arm_joint joint="joint5" axis="4" stream="${stream_position}"/>
+      <xacro:arm_joint joint="joint6" axis="5" stream="${stream_position}"/>
     </ros2_control>
   </xacro:macro>

File: wmx_r2_control/urdf/cr3a.wmx.urdf.xacro (robot description, xacro)
@@ -3,8 +3,13 @@
   <xacro:arg name="wmx_param_file"
              default="$(find wmx_r2_package)/config/cr3a_wmx_parameters.xml"/>
+  <!-- Export 'position' command interfaces and stream them through the WMX3
+       cyclic buffer. Set false for the previous feedback-only behaviour; see
+       cr3a.wmx.ros2_control.xacro. -->
+  <xacro:arg name="stream_position" default="true"/>
   <xacro:include filename="$(find movensys_manipulator_description)/urdf/dobot_cr3a/movensys_manipulator.xacro"/>
   <xacro:include filename="$(find wmx_r2_control)/urdf/cr3a.wmx.ros2_control.xacro"/>
   <xacro:movensys_manipulator_arm_wmx_r2_control
       name="WmxManipulatorArmSystem"
-      wmx_param_file="$(arg wmx_param_file)"/>
+      wmx_param_file="$(arg wmx_param_file)"
+      stream_position="$(arg stream_position)"/>
 </robot>
